File: RGBchristmasStar.sch (KiCad schematic (older format))
At the start: 45 parts, among them U1 WeMos_D1_mini

Commit message: created new footprints
Parts:
- D1, D10, D11, D12, D13, D14, D15, D16, D17, D18, D19, D2, D20, D21, D22, D3, D4, D5, D6, D7, D8, D9: footprint LED_SMD:LED_WS2812B_PLCC4_5.0x5.0mm_P3.2mm -> lib_fp:WS2812B-Mini; JLCPCB Part # (none) -> C114583
- U1: footprint Module:WEMOS_D1_mini_light -> lib_fp:WEMOS_D1_mini_light_SMD_header
